File: eDNA-SingleBoard-V3.brd (EAGLE design)
At the start: 107 x 70 mm, 89 parts, among them J1 PJS008U-3000-0, Q1 DMN65D8L-7, Q2 DMN65D8L-7, Q3 DMN65D8L-7, U1 TXS0108EPWR

Commit message: Updated SCH and PCB
Parts:
- removed TEST-GND, TEST-GND1: (no value), adafruit:1X01
- added 12V, 3V, 5V, GND, GND1: TPPAD1-13, testpad:P1-13
- added C1, C2: 100nF, resistor:C0805
- added J2: MEM2051-00-195-00-A, MEM2051-00-195-00-A:GCT_MEM2051-00-195-00-A
- added R22: 10K, adafruit:R0805
- moved R20 120.7 mm to (70.2, 5.59), turned to 90 degrees
- moved R19 119.1 mm to (72.8, 6.60), turned to 90 degrees
- moved C17 12.6 mm to (3.94, 45.7), turned to 180 degrees
- moved U1 3.95 mm to (64.6, 8.00)
- moved D3 0.64 mm to (62.7, 43.4)
- moved C3 0.64 mm to (22.7, 28.2)
- moved C18 0.63 mm to (24.1, 42.9)
- moved I2C_5V 0.63 mm to (53.8, 14.9)
- moved RTC 0.63 mm to (22.9, 35.6)
- moved COUT 0.38 mm to (63.1, 39.6)
Connections:
- removed net 3VRAIL: C17.1, J1.4
- net +12V: now also 12V.TP
- net +3V3: now also 3V.TP, C17.1, C2.1, J1.4, J2.4, R22.2, U1.10
- net +5V: now also 5V.TP, C1.1
- net 5V_SCL: now also U1.14; no longer U1.15
- net 5V_SDA: now also U1.15; no longer U1.14
- net CS: now also J2.2
- net DGND: now also C1.2, C2.2, GND.TP, GND1.TP, J2.6, R22.1; no longer TEST-GND.1, TEST-GND1.1
- net DI: now also J2.3
- net DO: now also J2.7
- net SCK: now also J2.5
- net SCL: now also U1.7; no longer U1.6
- net SDA: now also U1.6; no longer U1.7
Routing:
- net +5V: track 0.00 -> 178.2 mm, vias 0 -> 6
- net +3V3: track 0.00 -> 133.0 mm
- net SDA: track 0.00 -> 103.2 mm, vias 0 -> 3
- net SCL: track 0.00 -> 91.4 mm, vias 0 -> 1
- net HB_IN2: track 0.00 -> 72.4 mm, vias 0 -> 2
- net HB_IN1: track 0.00 -> 67.2 mm, vias 0 -> 2
- net T_SCK: track 0.00 -> 63.3 mm, vias 0 -> 5
- net SHUTDOWN: track 0.00 -> 62.8 mm, vias 0 -> 2
- net T_RCK: track 0.00 -> 61.5 mm, vias 0 -> 5
- net RTC_INT: track 0.00 -> 58.7 mm, vias 0 -> 1
- net SHIFT_LATCH: track 0.00 -> 48.0 mm, vias 0 -> 1
- net SENSOR2: track 0.00 -> 45.9 mm
- net SCK: track 0.00 -> 45.0 mm, vias 0 -> 1
- net SHIFT_CLK: track 0.00 -> 44.6 mm, vias 0 -> 1
- net SENSOR1: track 0.00 -> 44.2 mm
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- added copper zone on layer 1, net +12V
- added copper zone on layer 16, net +12V
- added copper zone on layer 1, net +12V_NON_PROTECT
- added copper zone on layer 1, net 12V_IN
- added copper zone on layer 1, net 5V_MCU
- added copper zone on layer 1, net N$10
- added copper zone on layer 1, net N$12
- added copper zone on layer 1, net N$15
- added copper zone on layer 1, net N$16
- added copper zone on layer 1, net N$17
- added copper zone on layer 1, net N$19
- added copper zone on layer 1, net N$3
