File: eDNA-SingleBoard-V3.sch (EAGLE design)
At the start: 86 parts, among them J1 PJS008U-3000-0, Q1 DMN65D8L-7, Q2 DMN65D8L-7, Q3 DMN65D8L-7

Commit message: Updated Schematic
Parts:
- removed B1: SPARKFUN_LOGIC_LEVEL_CONVERTER, SparkFun-Boards:SPARKFUN_LOGIC_LEVEL_CONVERTER
- removed I2C1, I2C2, I2C3: DF51-4POS, HiroseConnectors:DF51-4POS
- added I2C_3V, I2C_5V, PRESSURE: DF51-4POS, HiroseConnectors:DF51-4POS
- added R19, R20: 10K, rcl:R-US_R0805
- added U1: TXS0108EPWR, TXS0108EPWR:TXS0108EPWR
Connections:
- removed net 12VRAIL: PMOS3.D
- removed net 5VRAIL: PMOS1.D
- new net 12V_IN: CIN1.1, CIN2.1, D4.C, D5.C, L3.1, NMOS.D, PMOS3.S, R8.2, U$7.OUT
- new net 3V_MCU: MS1.3V, PMOS2.S, R18.2
- new net 5V_MCU: COUT.1, L1.2, MS1.USB, PMOS1.S, R11.2, R7.2, VREG.FB
- new net 5V_SCL: I2C_5V.P4, R20.2, U1.B5
- new net 5V_SDA: I2C_5V.P3, R19.2, U1.B6
- net +12V: now also PMOS3.D; no longer CIN1.1, CIN2.1, D4.C, D5.C, L3.1, NMOS.D, PMOS3.S, R8.2, U$7.OUT
- net +3V3: now also I2C_3V.P1, PMOS2.D, PRESSURE.P1, U1.VCCA; no longer B1.LV, I2C1.P1, I2C2.P1, I2C3.P1, MS1.3V, PMOS2.S, R18.2
- net +5V: now also I2C_5V.P1, PMOS1.D, R19.1, R20.1, U1.VCCB; no longer B1.HV, COUT.1, L1.2, MS1.USB, PMOS1.S, R11.2, R7.2, VREG.FB
- net 3VRAIL: no longer PMOS2.D
- net DGND: now also C10.2, C11.-, C12.2, C13.2, C15.-, C16.2, C20.2, C7.2, C8.2, C9.2, DRV8871-2.GND, DRV8871-2.PGND, DRV8871.GND, DRV8871.PGND, I2C_3V.P2, I2C_5V.P2, NOTGATE1.GND, NOTGATE2.GND, PRESSURE.P2, R14.1, R15.1, TPIC0.10, TPIC0.11, TPIC0.19, TPIC0.GND, TPIC1.10, TPIC1.11, TPIC1.19, TPIC1.GND, TPIC2.10, TPIC2.11, TPIC2.19, TPIC2.GND, TPIC3.10, TPIC3.11, TPIC3.19, TPIC3.GND, U1.GND; no longer I2C1.P2, I2C2.P2, I2C3.P2
- net GND: no longer B1.GND, B1.GND@2, C10.2, C11.-, C12.2, C13.2, C15.-, C16.2, C20.2, C7.2, C8.2, C9.2, DRV8871-2.GND, DRV8871-2.PGND, DRV8871.GND, DRV8871.PGND, NOTGATE1.GND, NOTGATE2.GND, R14.1, R15.1, TPIC0.10, TPIC0.11, TPIC0.19, TPIC0.GND, TPIC1.10, TPIC1.11, TPIC1.19, TPIC1.GND, TPIC2.10, TPIC2.11, TPIC2.19, TPIC2.GND, TPIC3.10, TPIC3.11, TPIC3.19, TPIC3.GND
- net SCL: now also I2C_3V.P4, PRESSURE.P4, U1.A5; no longer I2C1.P4, I2C2.P4, I2C3.P4
- net SDA: now also I2C_3V.P3, PRESSURE.P3, U1.A6; no longer I2C1.P3, I2C2.P3, I2C3.P3
- net SHIFT_CLK: now also U1.A3; no longer B1.LV_RXO_2
- net SHIFT_DATA: now also U1.A1; no longer B1.LV_TXI_1
- net SHIFT_LATCH: now also U1.A2; no longer B1.LV_RXO_1
- net T_DATA: now also U1.B1; no longer B1.HV_TXO_1
- net T_RCK: now also U1.B2; no longer B1.HV_RXI_1
- net T_SCK: now also U1.B3; no longer B1.HV_RXI_2
Other:
- note removed: "Modify this circuit with Hypnos Power Cutoff Circuit"
- moved on the sheet: 0X76, ANALOG1, ANALOG2, B2, C10, C11, C12, C13, C14, C15, C17, C18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

Commit message: Updated Schematic and PCB Files
Parts:
- added R21: 100k, Resistor_Capacitor:WSLP1206R0500FEA
- C10, C12, C13, C16, C20, C5, C7, C8, C9: device resistor:C-USC1206 -> resistor:C-USC0805
- CBOOT, COUT: device rcl:C-USC1206 -> rcl:C-USC0805
- CIN, CIN1, CIN2: device rcl:C-USC1206K -> rcl:C-USC0805
- R11: device Resistor_Capacitor:WSLP1206R0500FEA -> resistor:R-US_R0805
- R12, R13: device adafruit:R-US_R1206 -> adafruit:R-US_R0805
- R14, R15, RGND: device rcl:R-US_R1206 -> rcl:R-US_R0805
Connections:
- new net N$12: R21.1, VREG.!SHDN
- net N$15: now also R21.2; no longer VREG.!SHDN
Other:
- note added: "Add the necessary components to the logic Converter"
- moved on the sheet: CBOOT, COUT, D3, L1, LED, LED1, P_MOS, R16, R17, R19, R20, R3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

Commit message: Updated SCH and PCB
Parts:
- removed TEST-GND, TEST-GND1: (no value), adafruit:PINHD-1X1
- added 12V, 3V, 5V, GND, GND1: TPPAD1-13, testpad:TPPAD1-13
- added C1, C2: 100nF, resistor:C-USC0805
- added J2: MEM2051-00-195-00-A, MEM2051-00-195-00-A:MEM2051-00-195-00-A
- added R22: 10K, adafruit:R-US_R0805
Connections:
- removed net 3VRAIL: C17.1, J1.VDD
- net +12V: now also 12V.TP
- net +3V3: now also 3V.TP, C17.1, C2.1, J1.VDD, J2.VDD, R22.2, U1.OE
- net +5V: now also 5V.TP, C1.1
- net 5V_SCL: now also U1.B6; no longer U1.B5
- net 5V_SDA: now also U1.B5; no longer U1.B6
- net CS: now also J2.DATA3/CD
- net DGND: now also C1.2, C2.2, GND.TP, GND1.TP, J2.VSS, R22.1; no longer TEST-GND.1, TEST-GND1.1
- net DI: now also J2.CMD
- net DO: now also J2.DATA0
- net SCK: now also J2.CLK
- net SCL: now also U1.A6; no longer U1.A5
- net SDA: now also U1.A5; no longer U1.A6
Other:
- note removed: "Add the necessary components to the logic Converter"
- moved on the sheet: C11, C12, C15, C17, DRV8871, J1, R14, U$4, U$5, U1
